File: hardware/LoRa_PCIe_GW_GPS.sch (KiCad schematic (older format))
At the start: 11 parts, among them Q600 NC, U600 ZOE-M8Q

Commit message: Added BOM for non GNSS variants. Few part numbers corrected in design.
Parts:
- U600: value ZOE-M8Q -> EVA-M8M-0
Changed lines of the file:
@@
 P 4675 3350
 F 0 "U600" H 3925 4375 60  0000 L BNN
-F 1 "ZOE-M8Q" H 3900 2150 60  0000 L BNN
+F 1 "EVA-M8M-0" H 3900 2150 60  0000 L BNN
 F 2 "LoRa_PCIe_GW:LGA43R65P9X9_700X700X116" H 5795 6750 60  0001 C CNN
 F 3 "https://www.u-blox.com/en/docs/UBX-16014189" H 5795 6750 60  0001 C CNN
