File: hardware/LoRa_PCIe_GW_Interface.sch (KiCad schematic (older format))
At the start: 41 parts, among them Q300 NC, U300 NC

Commit message: Updates according to Corecell_V3 Reference design.
Parts:
- added C305: NC, LoRa_PCIe_GW:ccer_603_smd_small, symbol LoRa_PCIe_GW-rescue:Cap-
- added C312: 100nF, LoRa_PCIe_GW:ccer_402_smd_small, symbol LoRa_PCIe_GW-rescue:Cap-
- added D301: NC, LoRa_PCIe_GW:SLP1006P2T, symbol LoRa_PCIe_GW-rescue:RClamp0531T-
- added FB301: NC, LoRa_PCIe_GW:rlc_402_smd_small, symbol LoRa_PCIe_GW-rescue:Ferrite_beads-
- added L300: NC, LoRa_PCIe_GW:IND_744232090, symbol LoRa_PCIe_GW-rescue:L_Core_Ferrite_Coupled
- added R300, R325, R327: NC, LoRa_PCIe_GW:rlc_201_smd_small, symbol LoRa_PCIe_GW-rescue:Resistor-
- C308: renamed from C300; value 10uF -> 47uF; Description 10µF ±10% 16V Ceramic Capacitor X5R 0603 (1608 Metric) -> Multilayer ceramic capacitors X5R ±20%, 6.3V; Part Number GRM188R61C106KAAL -> GRM188R60J476ME15D
- C309: value 100nF -> NC
- R306, R307, R312, R314, R315, R320, R322, R323: Description 100 Ohms ±1% 0.05W, 1/20W Chip Resistor 0201 (0603 Metric) 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 -> 1k Ohm ±5% 0.05W, 1/20W Chip Resistor 0201 (0603 Metric) - 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; Part Number CRCW0201100R -> CRCW02011K00JNED; Price[1k] 0.037 -> 0.073; Supplier Link https://www.digikey.com/en/products/detail/vishay-dale/CRCW0201100RFKED/1967973 -> https://www.digikey.com/en/products/detail/vishay-dale/CRCW02011K00JNED/1178450
- R330: value 100R -> 1k; Description 100 Ohms ±1% 0.05W, 1/20W Chip Resistor 0201 (0603 Metric) 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 -> 1k Ohm ±5% 0.05W, 1/20W Chip Resistor 0201 (0603 Metric) - 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; Part Number CRCW0201100R -> CRCW02011K00JNED; Price[1k] 0.037 -> 0.073; Supplier Link https://www.digikey.com/en/products/detail/vishay-dale/CRCW0201100RFKED/1967973 -> https://www.digikey.com/en/products/detail/vishay-dale/CRCW02011K00JNED/1178450
- renumbered R300 to R326
Connections:
- net labels added: MCU_BOOT0, SX1302_GPIO_8, SX1302_RESET_HOST, VCC5V_IN
- wire segments 179 -> 201
- no-connect marks 11 -> 8
Other:
- moved on the sheet: C309, C310, C311, D302, FB302, R308, R309, R322, R323
