File: hardware/LoRa_PCIe_GW_Power.sch (KiCad schematic (older format))
At the start: 46 parts, among them U201 3V3, U202 TPS62242DRV, U203 3V3, U204 STTS751, U205 NCP176BMX330TCG, U206 3V3

Commit message: Updates according to Corecell_V3 Reference design.
Parts:
- added C200: 1uF, LoRa_PCIe_GW:ccer_402_smd_small, symbol LoRa_PCIe_GW-rescue:Cap-
- added C205, C211: NC, LoRa_PCIe_GW:ccer_603_smd_small, symbol LoRa_PCIe_GW-rescue:Cap-
- added C209, C215: NC, LoRa_PCIe_GW:ccer_402_smd_small, symbol LoRa_PCIe_GW-rescue:Cap-
- added C214: NC, LoRa_PCIe_GW:ccer_201_smd_small, symbol LoRa_PCIe_GW-rescue:Cap-
- added FB203, FB206: NC, LoRa_PCIe_GW:rlc_402_smd_small, symbol LoRa_PCIe_GW-rescue:Ferrite_beads-
- added L201: NC, LoRa_PCIe_GW:LQM2HPN2R2MJ0L, symbol LoRa_PCIe_GW-rescue:Inductor-
- added R200, R207: 0R, LoRa_PCIe_GW:rlc_201_smd_small, symbol LoRa_PCIe_GW-rescue:Resistor-
- added R209, R210, R211, R212, R213: NC, LoRa_PCIe_GW:rlc_201_smd_small, symbol LoRa_PCIe_GW-rescue:Resistor-
- added R222: NC, LoRa_PCIe_GW:rlc_402_smd_small, symbol LoRa_PCIe_GW-rescue:Resistor-
- added U200: NC, LoRa_PCIe_GW:DSBGA-4, symbol LoRa_PCIe_GW-rescue:TPS22908
- added U207: NC, LoRa_PCIe_GW:DRV0006A_V, symbol LoRa_PCIe_GW-rescue:TI-TPS62242DRV6-1600X1000TP-
- C208, C220, C221: footprint LoRa_PCIe_GW:ccer_201_smd_small -> LoRa_PCIe_GW:ccer_402_smd_small; Description 0.1µF ±10% 16V Ceramic Capacitor X7S 0201 (0603 Metric) -> Multilayer ceramic capacitors X7R ±10%, 16V; Part Number GRM033C71C104KE14D -> GMD155R71C104KA11; Supplier Link https://www.digikey.com/en/products/detail/murata-electronics/GRM033C71C104KE14D/5027472 -> https://www.digikey.com/en/products/detail/murata-electronics/GMD155R71C104KA11D/10696609
- R201, R205: value 10k -> 47k; Description 10 kOhms ±1% 0.05W, 1/20W Chip Resistor 0201 Thick Film -> 47 kOhms ±5% 0.05W, 1/20W Chip Resistor 0201 Thick Film; Part Number CRCW020110K0 -> CRCW020147K0; Price[1k] 0.037 -> 0.039; Supplier Link https://www.digikey.com/en/products/detail/vishay-dale/CRCW020110K0FKED/1967989 -> https://www.digikey.com/en/products/detail/vishay-dale/CRCW020147K0FKED/1968131
- R204: footprint LoRa_PCIe_GW:rlc_402_smd_small -> LoRa_PCIe_GW:rlc_201_smd_small; Description CRCW04020000ZSTD -> 0 Ohms Jumper 0.05W, 1/20W Chip Resistor 0201 (0603 Metric)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; Part Number CRCW04020000ZSTD -> CRCW02010000Z0ED; Price[1k] 0.014 -> 0.006; Supplier Link https://www.digikey.com/en/products/detail/vishay-dale/CRCW04020000ZSTD/1226552 -> https://www.digikey.com/en/products/detail/vishay-dale/CRCW02010000Z0ED/1178434?s=N4IgTCBcDaIMICU4HUAMZUEZU9QLVQFEAREAXQF8g
- R208: Description 1 kOhms ±5% 0.05W, 1/20W Chip Resistor 0201 (0603 Metric) T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 -> 1k Ohm ±5% 0.05W, 1/20W Chip Resistor 0201 (0603 Metric) - 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; Price[1k] 0.007 -> 0.073; Supplier Link https://www.digikey.com/en/products/detail/vishay-dale/CRCW02011K00JNED/1178450?s=N4IgTCBcDaIMICU4HUAMZUEZMGlWoCkA5AUQBEQBdAXyA -> https://www.digikey.com/en/products/detail/vishay-dale/CRCW02011K00JNED/1178450
- R215: renamed from R202; Label Other -> (none)
Connections:
- net GND: now also C200.2, C205.2, C209.2, C211.2, C215.2, R210.1, R212.1, U200.B1 (GND), U207.6 (GND), U207.7 (PP)
- net SX1302_CSD: now also R204.1, R207.1; no longer U205.4 (EN)
- net VCCCORE12: now also R200.1
- net VCC_FEM: now also FB206.2
- net VCC_FEM1: now also R222.1
- net VCC_MAIN: now also C205.1, R209.1, U207.5 (VIN); no longer R204.2, R215.2, U201.3 (EN)
- net VDD_RADIO: now also FB203.2
- net at C213.1, FB205.1, U203.1 (OUT): no longer R204.1
- net at C202.1, FB207.1, R215.1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: now also U200.A1 (VOUT)
- new net: C200.1, R200.2, U200.B2 (ON), U201.3 (EN)
- new net: L201.1, U207.1 (SW)
- new net: R209.2, R210.2, R213.2, U207.2 (MODE)
- new net: C214.1, R211.1, R212.2, U207.3 (FB)
- new net: C211.1, C214.2, FB206.1, L201.2, R211.2
- new net SX1302_PS_EN: R213.1
- new net U205_EN: R207.2, U205.4 (EN)
- new net U206_EN: R204.2, U207.4 (EN)
- new net VCC3V3_IN: C209.1, C215.1, FB203.1, R215.2, R222.2, U200.A2 (VIN)
Other:
- moved on the sheet: C201, C202, C203, C204, C206, C207, C208, C212, C213, C220, C221, C222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

Commit message: Signed-off-by: mmilann <milan@nebra.com>
Parts:
- added C210, C216: 100nF, LoRa_PCIe_GW:ccer_402_smd_small, symbol LoRa_PCIe_GW-rescue:Cap-
- added C231: 22pF, LoRa_PCIe_GW:ccer_201_smd_small, symbol LoRa_PCIe_GW-rescue:Cap-
- added R231, R232: 182K, LoRa_PCIe_GW:rlc_201_smd_small, symbol LoRa_PCIe_GW-rescue:Resistor-
- C206: value 4.7uF -> 47uF; Description 4.7µF ±10% 16V Ceramic Capacitor X5R 0603 (1608 Metric) -> Multilayer ceramic capacitors X5R ±20%, 6.3V; Part Number GRM188R61C475KAAJD -> GRM188R60J476ME15D; Price[1k] 0.089 -> 0.1; Supplier Link https://www.digikey.com/en/products/detail/murata-electronics/GRM188R61C475KAAJD/5027566 -> https://www.digikey.com/en/products/detail/murata-electronics/GRM188R61C106KAALJ/4905339
- C207, C212: value 10uF -> NC
- C213: value 4.7uF -> NC
- C215: value NC -> 47uF; footprint LoRa_PCIe_GW:ccer_402_smd_small -> LoRa_PCIe_GW:ccer_603_smd_small; Description 4.7µF ±20% 6.3V Ceramic Capacitor X5R 0402 (1005 Metric) -> Multilayer ceramic capacitors X5R ±20%, 6.3V; Part Number GRM155R60J475ME47D -> GRM188R60J476ME15D; Price[1k] 0.089 -> 0.1; Supplier Link https://www.digikey.com/en/products/detail/murata-electronics/GRM155R60J475ME47D/3694656 -> https://www.digikey.com/en/products/detail/murata-electronics/GRM188R61C106KAALJ/4905339
- C222: value 2.2uF -> NC
- C223: value 100nF -> NC
- C225: value 1uF -> NC
- FB203: value NC -> Ferrite beads
- FB205: value Ferrite beads -> NC
- R201: value 47k -> 47K
- R205: value 47k -> NC
- R207: value 0R -> NC
- R221, R222: value NC -> 0R
- U201: Alternatives (none) -> NCP4586DMU33TCG; Description Linear Voltage Regulator IC Positive Fixed 1 Output 150mA 4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 -> Linear Voltage Regulator IC Positive Fixed 1 Output 300mA 4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; Part Number NCP103AMX330TCG -> NCP114AMX330TCG; Price[1k] 0.097 -> 0.079; Supplier Link https://www.digikey.com/en/products/detail/on-semiconductor/NCP103AMX330TCG/5022526 -> https://www.digikey.com/en/products/detail/on-semiconductor/NCP114AMX330TBG/6166731
- U202: value TPS62242DRV -> TPS62260DRV; Alternative1 (none) -> SY20183LDEC; Description Buck Switching Regulator IC Positive Fixed 1.2V 1 Output 30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 -> Buck Switching Regulator IC Positive Adjustable 0.6V 1 Outp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; Part Number TPS62242DRV -> TPS62260DRV; Price[1k] 0.53 -> 0.85; Supplier Link https://www.digikey.com/en/products/detail/texas-instruments/TPS62242DRVR/1908036 -> https://www.digikey.com/en/products/detail/texas-instruments/TPS62260DRVR/1908045
- U203, U206: value 3V3 -> NC
- U204: value STTS751 -> NC
- U205: value NCP176BMX330TCG -> NC
Connections:
- net GND: now also C210.1, C216.1, R232.1
- net VCC3V3_IN: now also R221.2, C216.2
- net VCC_FEM1: now also C210.2
- net VCC_MAIN: no longer R221.2
- net at C203.1, FB208.1, L200.2: now also C231.2, R231.2; no longer U202.3 (FB)
- new net: C231.1, R231.1, R232.2, U202.3 (FB)
Other:
- moved on the sheet: C203, C204, L200, U202
