File: hardware/LoRa_PCIe_GW_RF.kicad_sch (KiCad schematic)
At the start: 94 parts, among them U700 NC, U800 SX1250, U801 SAW Filter, U802 SKY66423-11, U803 SAW Filter, U805 SAW Filter, U900 SX1250, Y800 TCXO

Commit message: Fixed ERC and Schematic to Layout parity errors.
Other:
- note added: "TVS Diode"
Changed lines of the file:
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@@
   (junction (at 390.525 235.585) (diameter 0) (color 0 0 0 0)
   )
+  (junction (at 133.985 153.67) (diameter 0) (color 0 0 0 0)
+  )
   (junction (at 453.39 123.825) (diameter 0) (color 0 0 0 0)
   )
@@
   (junction (at 268.605 352.425) (diameter 0) (color 0 0 0 0)
   )
+  (junction (at 162.56 316.23) (diameter 0) (color 0 0 0 0)
+  )
   (junction (at 245.11 349.25) (diameter 0) (color 0 0 0 0)
   )
+  (junction (at 130.81 351.155) (diameter 0) (color 0 0 0 0)
+  )
   (junction (at 300.99 187.96) (diameter 0) (color 0 0 0 0)
   )
@@
   (junction (at 157.48 316.23) (diameter 0) (color 0 0 0 0)
   )
+  (junction (at 410.845 134.62) (diameter 0) (color 0 0 0 0)
+  )
   (junction (at 163.195 348.615) (diameter 0) (color 0 0 0 0)
   )
@@
   (junction (at 300.99 243.84) (diameter 0) (color 0 0 0 0)
   )
+  (junction (at 134.62 257.81) (diameter 0) (color 0 0 0 0)
+  )
   (junction (at 410.845 119.38) (diameter 0) (color 0 0 0 0)
   )
@@
     (stroke (width 0) (type default) (color 0 0 0 0))
   )
-  (wire (pts (xy 142.875 257.81) (xy 127.635 257.81))
+  (wire (pts (xy 142.875 257.81) (xy 134.62 257.81))
     (stroke (width 0) (type default) (color 0 0 0 0))
   )
@@
     (stroke (width 0) (type default) (color 0 0 0 0))
   )
-  (wire (pts (xy 137.795 351.155) (xy 123.825 351.155))
+  (wire (pts (xy 137.795 351.155) (xy 130.81 351.155))
     (stroke (width 0) (type default) (color 0 0 0 0))
   )
@@
     (stroke (width 0) (type default) (color 0 0 0 0))
   )
-  (wire (pts (xy 140.97 153.67) (xy 127.635 153.67))
+  (wire (pts (xy 133.985 153.67) (xy 127.635 153.67))
+    (stroke (width 0) (type default) (color 0 0 0 0))
+  )
+  (wire (pts (xy 140.97 153.67) (xy 133.985 153.67))
     (stroke (width 0) (type default) (color 0 0 0 0))
   )
@@
     (stroke (width 0) (type default) (color 0 0 0 0))
   )
+  (wire (pts (xy 130.81 351.155) (xy 123.825 351.155))
+    (stroke (width 0) (type default) (color 0 0 0 0))
+  )
   (wire (pts (xy 415.925 196.215) (xy 415.925 185.42))
     (stroke (width 0) (type default) (color 0 0 0 0))
@@
     (stroke (width 0) (type default) (color 0 0 0 0))
   )
+  (wire (pts (xy 134.62 257.81) (xy 127.635 257.81))
+    (stroke (width 0) (type default) (color 0 0 0 0))
+  )
   (wire (pts (xy 529.59 167.64) (xy 523.24 167.64))
     (stroke (width 0) (type default) (color 0 0 0 0))
@@
     (stroke (width 0) (type default) (color 0 0 0 0))
   )
+  (text "TVS Diode" (at 520.065 179.705 90)
+    (effects (font (size 1.27 1.27)) (justify left bottom))
+  )
   (text "See LoRa_Reference_Clock_Selection_V1.1 for recommended osc"
     (at 46.355 91.567 0)
@@
     (effects (font (size 1.524 1.524)) (justify left bottom))
   )
-  (label "TVS diode" (at 520.7 181.61 90)
-    (effects (font (size 1.778 1.778)) (justify left bottom))
-  )
   (label "TX_RF3" (at 271.78 121.92 0)
     (effects (font (size 1.27 1.27)) (justify left bottom))
@@
       (effects (font (size 1.524 1.524)) (justify right top))
     )
-    (property "Value" "1.2nH" (id 1) (at 407.67 133.35 90))
+    (property "Value" "1.2nH" (id 1) (at 412.115 127 0))
     (property "Footprint" "LoRa_PCIe_GW:rlc_402_smd_small" (id 2) (at 410.845 134.62 0)
       (effects (font (size 1.27 1.27)) hide)
@@
       (effects (font (size 1.27 1.27)) hide)
     )
+    (pin "1")
+  )
+  (symbol (lib_id "power:PWR_FLAG") (at 134.62 257.81 0) (unit 1)
+    (in_bom yes) (on_board yes) (fields_autoplaced)
+    (property "Reference" "#FLG0113" (id 0) (at 134.62 255.905 0)
+      (effects (font (size 1.27 1.27)) hide)
+    )
+    (property "Value" "PWR_FLAG" (id 1) (at 134.62 254.2342 0))
+    (property "Footprint" "" (id 2) (at 134.62 257.81 0)
+      (effects (font (size 1.27 1.27)) hide)
+    )
+    (property "Datasheet" "~" (id 3) (at 134.62 257.81 0)
+      (effects (font (size 1.27 1.27)) hide)
+    )
+    (pin "1")
+  )
+  (symbol (lib_id "power:PWR_FLAG") (at 410.845 134.62 90) (unit 1)
+    (in_bom yes) (on_board yes) (fields_autoplaced)
+    (property "Reference" "#FLG0111" (id 0) (at 408.94 134.62 0)
+      (effects (font (size 1.27 1.27)) hide)
+    )
+    (property "Value" "PWR_FLAG" (id 1) (at 407.6701 135.0538 90)
+      (effects (font (size 1.27 1.27)) (justify left))
+    )
+    (property "Footprint" "" (id 2) (at 410.845 134.62 0)
+      (effects (font (size 1.27 1.27)) hide)
+    )
+    (property "Datasheet" "~" (id 3) (at 410.845 134.62 0)
+      (effects (font (size 1.27 1.27)) hide)
+    )
+    (pin "1")
+  )
+  (symbol (lib_id "power:PWR_FLAG") (at 133.985 153.67 0) (unit 1)
+    (in_bom yes) (on_board yes) (fields_autoplaced)
+    (property "Reference" "#FLG0112" (id 0) (at 133.985 151.765 0)
+      (effects (font (size 1.27 1.27)) hide)
+    )
+    (property "Value" "PWR_FLAG" (id 1) (at 133.985 150.0942 0))
+    (property "Footprint" "" (id 2) (at 133.985 153.67 0)
+      (effects (font (size 1.27 1.27)) hide)
+    )
+    (property "Datasheet" "~" (id 3) (at 133.985 153.67 0)
+      (effects (font (size 1.27 1.27)) hide)
+    )
+    (pin "1")
+  )
+  (symbol (lib_id "power:PWR_FLAG") (at 130.81 351.155 0) (unit 1)
+    (in_bom yes) (on_board yes) (fields_autoplaced)
+    (property "Reference" "#FLG0110" (id 0) (at 130.81 349.25 0)
+      (effects (font (size 1.27 1.27)) hide)
+    )
+    (property "Value" "PWR_FLAG" (id 1) (at 130.81 347.5792 0))
+    (property "Footprint" "" (id 2) (at 130.81 351.155 0)
+      (effects (font (size 1.27 1.27)) hide)
+    )
+    (property "Datasheet" "~" (id 3) (at 130.81 351.155 0)
+      (effects (font (size 1.27 1.27)) hide)
+    )
+    (pin "1")
+  )
+  (symbol (lib_id "power:PWR_FLAG") (at 162.56 316.23 0) (unit 1)
+    (in_bom yes) (on_board yes) (fields_autoplaced)
+    (property "Reference" "#FLG0109" (id 0) (at 162.56 314.325 0)
+      (effects (font (size 1.27 1.27)) hide)
+    )
+    (property "Value" "PWR_FLAG" (id 1) (at 164.211 315.3938 0)
+      (effects (font (size 1.27 1.27)) (justify left))
+    )
+    (property "Footprint" "" (id 2) (at 162.56 316.23 0)
+      (effects (font (size 1.27 1.27)) hide)
+    )
+    (property "Datasheet" "~" (id 3) (at 162.56 316.23 0)
+      (effects (font (size 1.27 1.27)) hide)
+    )
